Commit message: 2nd commit

File: urdf/6dof_mani.urdf (robot description, URDF)
Before this commit: robot 6dof_mani, 10 links, 9 joints
Links:
- added link world
Joints:
- added joint fixed_joint: type fixed, parent world, child base_link, origin xyz=0 0 0 rpy=0 0 0
- joint Revolute_1: limit lower=-1.570796 upper=1.570796 effort=100 velocity=100 -> lower=-3.141593 upper=3.141593 effort=100 velocity=100
- joint Revolute_2: limit lower=-1.570796 upper=1.570796 effort=100 velocity=100 -> lower=-3.141593 upper=3.141593 effort=100 velocity=100
- joint Revolute_3: limit lower=-3.141593 upper=0.0 effort=100 velocity=100 -> lower=-4.71 upper=1.2 effort=100 velocity=100
- joint Revolute_4: limit lower=-1.570796 upper=1.570796 effort=100 velocity=100 -> lower=-3.141593 upper=3.141593 effort=100 velocity=100
- joint Revolute_5: limit lower=-1.570796 upper=1.570796 effort=100 velocity=100 -> lower=-3.141593 upper=3.141593 effort=100 velocity=100
- joint Revolute_6: limit lower=-1.570796 upper=1.570796 effort=100 velocity=100 -> lower=-3.141593 upper=3.141593 effort=100 velocity=100

File: urdf/6dof_mani.xacro (robot description, xacro)
@@ -4,4 +4,5 @@
   <xacro:include filename="/home/ydg/mani_ws/src/mani/urdf/6dof_mani.gazebo" />
   <xacro:include filename="/home/ydg/mani_ws/src/mani/urdf/6dof_mani.trans" />
+<link name="world"/>
 <link name="base_link">
   <inertial>
@@ -24,4 +25,9 @@
   </collision>
 </link>
+<joint name="fixed_joint" type="fixed">
+  <parent link="world"/>
+  <child link="base_link"/>
+  <origin xyz="0 0 0" rpy="0 0 0"/>
+</joint>
 <link name="link_8_1">
   <inertial>
@@ -223,5 +229,5 @@
   <child link="link_7_1"/>
   <axis xyz="0.0 0.0 -1.0"/>
-  <limit upper="1.570796" lower="-1.570796" effort="100" velocity="100"/>
+  <limit upper="3.141593" lower="-3.141593" effort="100" velocity="100"/>
 </joint>
 <joint name="Revolute_5" type="revolute">
@@ -230,5 +236,5 @@
   <child link="link_6_1"/>
   <axis xyz="-1.0 0.0 0.0"/>
-  <limit upper="1.570796" lower="-1.570796" effort="100" velocity="100"/>
+  <limit upper="3.141593" lower="-3.141593" effort="100" velocity="100"/>
 </joint>
 <joint name="Revolute_4" type="revolute">
@@ -237,5 +243,5 @@
   <child link="link_5_1"/>
   <axis xyz="0.0 0.0 -1.0"/>
-  <limit upper="1.570796" lower="-1.570796" effort="100" velocity="100"/>
+  <limit upper="3.141593" lower="-3.141593" effort="100" velocity="100"/>
 </joint>
 <joint name="Revolute_3" type="revolute">
@@ -244,5 +250,5 @@
   <child link="link_4_1"/>
   <axis xyz="-1.0 0.0 0.0"/>
-  <limit upper="0.0" lower="-3.141593" effort="100" velocity="100"/>
+  <limit upper="1.2" lower="-4.71" effort="100" velocity="100"/>
 </joint>
 <joint name="Rigid_7" type="fixed">
@@ -256,5 +262,5 @@
   <child link="link_2_1"/>
   <axis xyz="1.0 0.0 0.0"/>
-  <limit upper="1.570796" lower="-1.570796" effort="100" velocity="100"/>
+  <limit upper="3.141593" lower="-3.141593" effort="100" velocity="100"/>
 </joint>
 <joint name="Revolute_1" type="revolute">
@@ -263,52 +269,45 @@
   <child link="link_1_1"/>
   <axis xyz="0.0 0.0 1.0"/>
-  <limit upper="1.570796" lower="-1.570796" effort="100" velocity="100"/>
+  <limit upper="3.141593" lower="-3.141593" effort="100" velocity="100"/>
 </joint>
 <ros2_control name="mani_ros2_control" type="system">
   <hardware>
-      <!-- By default, set up controllers for simulation. This won't work on real hardware -->
-      <plugin>gazebo_ros2_control/GazeboSystem</plugin>
+    <plugin>gazebo_ros2_control/GazeboSystem</plugin>
   </hardware>
   <joint name="Revolute_1">
-      <command_interface name="position"/>
-      <state_interface name="position">
-        <param name="initial_value">0.0</param>
-      </state_interface>
-      <state_interface name="velocity"/>
+    <command_interface name="position"/>
+    <state_interface name="position"/>
+    <state_interface name="velocity"/>
+    <initial_position>0.0</initial_position>
   </joint>
   <joint name="Revolute_2">
-      <command_interface name="position"/>
-      <state_interface name="position">
-        <param name="initial_value">0.0</param>
-      </state_interface>
-      <state_interface name="velocity"/>
+    <command_interface name="position"/>
+    <state_interface name="position"/>
+    <state_interface name="velocity"/>
+    <initial_position>0.0</initial_position>
   </joint>
   <joint name="Revolute_3">
-      <command_interface name="position"/>
-      <state_interface name="position">
-        <param name="initial_value">0.0</param>
-      </state_interface>
-      <state_interface name="velocity"/>
+    <command_interface name="position"/>
+    <state_interface name="position"/>
+    <state_interface name="velocity"/>
+    <initial_position>-1.57</initial_position>
   </joint>
   <joint name="Revolute_4">
-      <command_interface name="position"/>
-      <state_interface name="position">
-        <param name="initial_value">0.0</param>
-      </state_interface>
-      <state_interface name="velocity"/>
+    <command_interface name="position"/>
+    <state_interface name="position"/>
+    <state_interface name="velocity"/>
+    <initial_position>0.0</initial_position>
   </joint>
   <joint name="Revolute_5">
-      <command_interface name="position"/>
-      <state_interface name="position">
-        <param name="initial_value">0.0</param>
-      </state_interface>
-      <state_interface name="velocity"/>
+    <command_interface name="position"/>
+    <state_interface name="position"/>
+    <state_interface name="velocity"/>
+    <initial_position>0.0</initial_position>
   </joint>
   <joint name="Revolute_6">
-      <command_interface name="position"/>
-      <state_interface name="position">
-        <param name="initial_value">0.0</param>
-      </state_interface>
-      <state_interface name="velocity"/>
+    <command_interface name="position"/>
+    <state_interface name="position"/>
+    <state_interface name="velocity"/>
+    <initial_position>0.0</initial_position>
   </joint>
 </ros2_control>

File: urdf/materials.xacro (robot description, xacro)
@@ -4,3 +4,6 @@
   <color rgba="0.700 0.700 0.700 1.000"/>
 </material>
+<material name="white">
+  <color rgba="1.00 1.00 1.00 1.000"/>
+</material>
 </robot>

Commit message: Orientation Error Fixed

File: urdf/6dof_mani.urdf (robot description, URDF)
Before this commit: robot 6dof_mani, 11 links, 10 joints
Joints:
- joint Revolute_3: limit lower=-4.71 upper=1.2 effort=100 velocity=100 -> lower=-4.712389 upper=1.570796 effort=100 velocity=100
- joint Revolute_5: limit lower=-3.141593 upper=3.141593 effort=100 velocity=100 -> lower=-1.570796 upper=1.570796 effort=100 velocity=100
- joint Slider_1: limit lower=0.0 upper=0.025 effort=100 velocity=100 -> lower=0.0 upper=0.0 effort=100 velocity=100
- joint Slider_2: limit lower=-0.025 upper=0.0 effort=100 velocity=100 -> lower=0.0 upper=0.0 effort=100 velocity=100
- joint fixed_joint: origin xyz=0 0 0 rpy=0 0 0 -> xyz=0 0 0 rpy=0 0 -1.570796

File: urdf/6dof_mani.xacro (robot description, xacro)
@@ -28,5 +28,5 @@
   <parent link="world"/>
   <child link="base_link"/>
-  <origin xyz="0 0 0" rpy="0 0 0"/>
+  <origin xyz="0 0 0" rpy="0 0 -1.570796"/>
 </joint>
 <link name="link_8_1">
@@ -215,5 +215,6 @@
   <child link="link_8_1"/>
   <axis xyz="1.0 0.0 0.0"/>
-  <limit upper="0.025" lower="0.0" effort="100" velocity="100"/>
+  <limit upper="0.0" lower="0.0" effort="100" velocity="100"/>
+  <!--<limit upper="0.025" lower="0.0" effort="100" velocity="100"/>-->
 </joint>
 <joint name="Slider_2" type="prismatic">
@@ -222,5 +223,6 @@
   <child link="link_9_1"/>
   <axis xyz="1.0 0.0 0.0"/>
-  <limit upper="0.0" lower="-0.025" effort="100" velocity="100"/>
+  <limit upper="0.0" lower="0.0" effort="100" velocity="100"/>
+  <!--<limit upper="0.0" lower="-0.025" effort="100" velocity="100"/>-->
 </joint>
 <joint name="Revolute_6" type="revolute">
@@ -236,5 +238,5 @@
   <child link="link_6_1"/>
   <axis xyz="-1.0 0.0 0.0"/>
-  <limit upper="3.141593" lower="-3.141593" effort="100" velocity="100"/>
+  <limit upper="1.570796" lower="-1.570796" effort="100" velocity="100"/>
 </joint>
 <joint name="Revolute_4" type="revolute">
@@ -250,5 +252,5 @@
   <child link="link_4_1"/>
   <axis xyz="-1.0 0.0 0.0"/>
-  <limit upper="1.2" lower="-4.71" effort="100" velocity="100"/>
+  <limit upper="1.570796" lower="-4.712389" effort="100" velocity="100"/>
 </joint>
 <joint name="Rigid_7" type="fixed">
